File: PSU.kicad_pcb (KiCad board)
At the start: 4 copper layers, 100 x 100 mm, 182 parts, among them IC400 TLP185xSE, IC401 TLP185xSE, IC403 ACS71240, IC407 TLP185xSE, IC410 TLP185xSE, J200 09031967921, J400 XT60-Angled-F, J401 Conn_01x06_Pin, J800 USB_C_Receptacle_USB2.0_16P, Q400 AO3400A, Q401 HSBA8119, Q402 HSBA8119, Q403 HSBA8119, Q404 AO3400A, Q700 MMST3904, SW400 TL2243, SW401 Push SW, U100 W25Q128, U301 TPS563201DDCR, U302 CH334P, U400 STM32H750VBTx, U401 TPD2E2U06DCK, U402 TPD2E2U06DCK, U403 INA219AIDCNR, U404 ADS1115IDGS, U500 TJA1044GTK_3Z, U600 TJA1044GTK_3Z, U700 STM32F103CBTx, U801 FSUSB42UMX, X300 Q13FC1350000400, X400 X322512MSB4SI, Y700 8 MHz, Y900 12Mhz

Commit message: Change resistor
Parts:
- removed R711: 33kΩ, PCM_JLCPCB:R_0402
- added R434: 36kΩ, PCM_JLCPCB:R_0603, F.Cu at (133.4, 128.0)
- SW401: value Push SW -> ~
- moved R710 0.82 mm to (133.8, 126.9)
Routing:
- net Net-(Q700-B): track 4.94 -> 5.82 mm
- net GND: track 146.8 -> 146.2 mm
